File: Arduino/StandAlone/PCB2/ArduinoStandaloneUsbSwitch-V2.sch (EAGLE design)
At the start: 45 parts, among them U1 INA219AIDCNRSOIC, U2 LM3526M-L

Commit message: Tidied up, added notes.
Other:
- note added: "4 Port Version. Free pins: * A4, A5, A6, D0 * MISO, SCK, MOSI - Without LEDS: D6, D7, RX, TX"
- note added: "Adafruit TFT BoB Connection * Vin - NC * 3v3 -> 3v3 * Gnd -> GND * SCK -> SCK * MISO -> NC (Unless SD Card used then MISO) * MOSI -> MOSI * TFT_CS -> D7 (2 Port) * RESET -> D6 (2 Port) (Worst case, reset) * D/C -> A4 (2 and 4 port) * Card_CS -> NC * Lite -> NC -> Maybe PWM, Pull low for light off"
- moved on the sheet: C1, C2, C5, C6, C7, D1, D2, H1, H2, H3, H4, JP1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
