File: Arduino/StandAlone/PCB2/ArduinoStandaloneUsbSwitch-4Port.brd (EAGLE design)
At the start: 55 x 98.5 mm, 66 parts, among them U1 INA219AIDCNRSOIC, U2 LM3526M-L, U3 LM3526M-L, U4 ARDUINO_MKRFOX1200PROTOPADS

Commit message: Added component values during build.
Parts:
- C3: value 0.1u -> 0.1uF
- C5: value (none) -> 0.1uF
- C6: value (none) -> 1uF
Changed lines of the file:
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@@
 <attribute name="NAME" x="51.0275" y="82.4735" size="1.27" layer="26" ratio="10" rot="MR0"/>
 <attribute name="VALUE" x="48.349" y="81.905" size="1.27" layer="28" ratio="10" rot="MR90"/>
+<attribute name="FARNELL" value="1208851" x="50" y="80" size="1.778" layer="28" rot="MR90" display="off"/>
 </element>
 <element name="D2" library="SparkFun-LED" package="LED3MM" value="" x="50" y="70" smashed="yes" rot="MR90">
@@
 <attribute name="NAME" x="23.12" y="32.9" size="1.778" layer="26" font="vector" ratio="16" rot="MR0"/>
 <attribute name="NAME" x="9.88" y="32.91" size="0.8128" layer="25" font="vector" ratio="16"/>
+<attribute name="FARNELL" value="1177882" x="16.5" y="31" size="1.778" layer="27" rot="R270" display="off"/>
 </element>
 <element name="USB1" library="Tinamous" package="USB-A-VERTICAL" value="USB-NEW" x="38.5" y="31" locked="yes" smashed="yes" rot="R270">
@@
 <attribute name="NAME" x="41.414" y="32.925" size="0.8128" layer="25"/>
 <attribute name="VALUE" x="41.735" y="35.699" size="0.5" layer="27" rot="R90"/>
+<attribute name="FARNELL" value="1435952" x="41.684" y="35.64" size="1.778" layer="27" display="off"/>
 </element>
 <element name="R2" library="SparkFun-Resistors" package="0805" value="" x="14.2075" y="25.5695" smashed="yes" rot="R180">
@@
 <attribute name="PROD_ID" value=" SWCH-08441" x="5" y="80" size="1.778" layer="28" rot="MR270" display="off"/>
 <attribute name="NAME" x="5.9525" y="83.4925" size="1.27" layer="26" ratio="10" rot="MR0"/>
+<attribute name="FARNELL" value="2533101" x="5" y="80" size="1.778" layer="28" rot="MR270" display="off"/>
 </element>
 <element name="S2" library="SparkFun-Electromechanical" package="TACTILE-PTH" value="SWITCH-MOMENTARY-2PTH" x="5" y="70" smashed="yes" rot="MR270">
@@
 <element name="U1" library="INA219AIDCNR" package="SO08" value="INA219AIDCNRSOIC" x="39.425" y="42.365" smashed="yes" rot="R180">
 <attribute name="NAME" x="43.5525" y="43.635" size="0.8128" layer="25" rot="R180"/>
+<attribute name="FARNELL" value="2496402" x="39.425" y="42.365" size="1.778" layer="27" rot="R180" display="off"/>
 </element>
 <element name="U2" library="LM3256M-L" package="SOIC127P640X175-8N" value="LM3526M-L" x="27.52" y="38.0145" smashed="yes" rot="R270">
@@
 <attribute name="VALUE" x="23.368" y="77.5335" size="0.4064" layer="27" rot="R270"/>
 </element>
-<element name="C5" library="SparkFun-Capacitors" package="0805" value="" x="34.29" y="42.2275" smashed="yes">
+<element name="C5" library="SparkFun-Capacitors" package="0805" value="0.1uF" x="34.29" y="42.2275" smashed="yes">
 <attribute name="NAME" x="33.528" y="43.053" size="0.8128" layer="25"/>
 <attribute name="VALUE" x="33.274" y="40.8305" size="0.4064" layer="27"/>
 </element>
-<element name="C6" library="SparkFun-Capacitors" package="0805" value="" x="30.0195" y="74.359" smashed="yes" rot="R270">
+<element name="C6" library="SparkFun-Capacitors" package="0805" value="1uF" x="30.0195" y="74.359" smashed="yes" rot="R270">
 <attribute name="NAME" x="30.845" y="75.121" size="0.4064" layer="25" rot="R270"/>
 <attribute name="VALUE" x="28.6225" y="75.375" size="0.4064" layer="27" rot="R270"/>
@@
 <attribute name="VALUE" x="37.846" y="8.6995" size="0.4064" layer="27" rot="R180"/>
 </element>
-<element name="C3" library="SparkFun-Capacitors" package="0805" value="0.1u" x="32.1945" y="23.0505" smashed="yes">
+<element name="C3" library="SparkFun-Capacitors" package="0805" value="0.1uF" x="32.1945" y="23.0505" smashed="yes">
 <attribute name="NAME" x="32.7025" y="24.1935" size="0.8128" layer="25"/>
 <attribute name="VALUE" x="31.1785" y="21.6535" size="0.4064" layer="27"/>

Commit message: Updated device values.
Parts:
- R17, R18, R2, R29, R3, R30, R4, R5, R6, R7, R8, R9: value (none) -> DNP
- U4: value ARDUINO_MKRFOX1200PROTOPADS -> ARDUINO MKR Series
Changed lines of the file:
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@@
 <layer number="45" name="Holes" color="7" fill="1" visible="yes" active="yes"/>
 <layer number="46" name="Milling" color="3" fill="1" visible="yes" active="yes"/>
-<layer number="47" name="Measures" color="7" fill="1" visible="yes" active="yes"/>
+<layer number="47" name="Measures" color="7" fill="1" visible="no" active="yes"/>
 <layer number="48" name="Document" color="7" fill="1" visible="yes" active="yes"/>
 <layer number="49" name="Reference" color="7" fill="1" visible="yes" active="yes"/>
@@
 <attribute name="FARNELL" value="1435952" x="41.684" y="35.64" size="1.778" layer="27" display="off"/>
 </element>
-<element name="R2" library="SparkFun-Resistors" package="0805" value="" x="14.2075" y="25.5695" smashed="yes" rot="R180">
+<element name="R2" library="SparkFun-Resistors" package="0805" value="DNP" x="14.2075" y="25.5695" smashed="yes" rot="R180">
 <attribute name="NAME" x="14.9695" y="24.744" size="0.8128" layer="25" rot="R180"/>
 <attribute name="VALUE" x="15.2235" y="26.9665" size="0.4064" layer="27" rot="R180"/>
 </element>
-<element name="R3" library="SparkFun-Resistors" package="0805" value="" x="14.2075" y="22.5945" smashed="yes" rot="R180">
+<element name="R3" library="SparkFun-Resistors" package="0805" value="DNP" x="14.2075" y="22.5945" smashed="yes" rot="R180">
 <attribute name="NAME" x="14.9695" y="21.769" size="0.8128" layer="25" rot="R180"/>
 <attribute name="VALUE" x="15.2235" y="23.9915" size="0.4064" layer="27" rot="R180"/>
 </element>
-<element name="R4" library="SparkFun-Resistors" package="0805" value="" x="19.2875" y="25.5695" smashed="yes" rot="R180">
+<element name="R4" library="SparkFun-Resistors" package="0805" value="DNP" x="19.2875" y="25.5695" smashed="yes" rot="R180">
 <attribute name="NAME" x="20.0495" y="24.744" size="0.8128" layer="25" rot="R180"/>
 <attribute name="VALUE" x="20.3035" y="26.9665" size="0.4064" layer="27" rot="R180"/>
 </element>
-<element name="R5" library="SparkFun-Resistors" package="0805" value="" x="19.2875" y="22.5945" smashed="yes" rot="R180">
+<element name="R5" library="SparkFun-Resistors" package="0805" value="DNP" x="19.2875" y="22.5945" smashed="yes" rot="R180">
 <attribute name="NAME" x="20.0495" y="21.769" size="0.8128" layer="25" rot="R180"/>
 <attribute name="VALUE" x="20.3035" y="23.9915" size="0.4064" layer="27" rot="R180"/>
 </element>
-<element name="R6" library="SparkFun-Resistors" package="0805" value="" x="36.27" y="25.025" smashed="yes" rot="R180">
+<element name="R6" library="SparkFun-Resistors" package="0805" value="DNP" x="36.27" y="25.025" smashed="yes" rot="R180">
 <attribute name="NAME" x="37.032" y="24.1995" size="0.8128" layer="25" rot="R180"/>
 <attribute name="VALUE" x="37.286" y="26.422" size="0.4064" layer="27" rot="R180"/>
 </element>
-<element name="R7" library="SparkFun-Resistors" package="0805" value="" x="36.27" y="21.85" smashed="yes" rot="R180">
+<element name="R7" library="SparkFun-Resistors" package="0805" value="DNP" x="36.27" y="21.85" smashed="yes" rot="R180">
 <attribute name="NAME" x="37.032" y="21.0245" size="0.8128" layer="25" rot="R180"/>
 <attribute name="VALUE" x="37.286" y="23.247" size="0.4064" layer="27" rot="R180"/>
 </element>
-<element name="R8" library="SparkFun-Resistors" package="0805" value="" x="41.35" y="21.85" smashed="yes" rot="R180">
+<element name="R8" library="SparkFun-Resistors" package="0805" value="DNP" x="41.35" y="21.85" smashed="yes" rot="R180">
 <attribute name="NAME" x="42.112" y="21.0245" size="0.8128" layer="25" rot="R180"/>
 <attribute name="VALUE" x="42.366" y="23.247" size="0.4064" layer="27" rot="R180"/>
 </element>
-<element name="R9" library="SparkFun-Resistors" package="0805" value="" x="41.35" y="25.025" smashed="yes" rot="R180">
+<element name="R9" library="SparkFun-Resistors" package="0805" value="DNP" x="41.35" y="25.025" smashed="yes" rot="R180">
 <attribute name="NAME" x="42.112" y="24.1995" size="0.8128" layer="25" rot="R180"/>
 <attribute name="VALUE" x="42.366" y="26.422" size="0.4064" layer="27" rot="R180"/>
@@
 <attribute name="NAME" x="6.1025" y="73.58" size="1.27" layer="26" ratio="10" rot="MR0"/>
 </element>
-<element name="U4" library="Arduino" package="ARDUINO_MKRFOX1200_PROTOPADS" value="ARDUINO_MKRFOX1200PROTOPADS" x="14.605" y="36.195" locked="yes" smashed="yes"/>
+<element name="U4" library="Arduino" package="ARDUINO_MKRFOX1200_PROTOPADS" value="ARDUINO MKR Series" x="14.605" y="36.195" locked="yes" smashed="yes"/>
 <element name="U1" library="INA219AIDCNR" package="SO08" value="INA219AIDCNRSOIC" x="39.425" y="42.365" smashed="yes" rot="R180">
 <attribute name="NAME" x="43.5525" y="43.635" size="0.8128" layer="25" rot="R180"/>
@@
 <attribute name="VALUE" x="26.8605" y="32.766" size="0.4064" layer="27" rot="R270"/>
 </element>
-<element name="R29" library="SparkFun-Resistors" package="0805" value="" x="16.5" y="30.907" smashed="yes">
+<element name="R29" library="SparkFun-Resistors" package="0805" value="DNP" x="16.5" y="30.907" smashed="yes">
 <attribute name="NAME" x="15.738" y="31.7325" size="0.8128" layer="25"/>
 <attribute name="VALUE" x="15.484" y="29.51" size="0.4064" layer="27"/>
 </element>
-<element name="R30" library="SparkFun-Resistors" package="0805" value="" x="38.665" y="30.799" smashed="yes">
+<element name="R30" library="SparkFun-Resistors" package="0805" value="DNP" x="38.665" y="30.799" smashed="yes">
 <attribute name="NAME" x="37.903" y="31.6245" size="0.8128" layer="25"/>
 <attribute name="VALUE" x="37.649" y="29.402" size="0.4064" layer="27"/>
@@
 <attribute name="VALUE" x="42.418" y="94.107" size="0.4064" layer="27" rot="R270"/>
 </element>
-<element name="R17" library="SparkFun-Resistors" package="0805" value="" x="16.3195" y="14.6685" smashed="yes" rot="R180">
+<element name="R17" library="SparkFun-Resistors" package="0805" value="DNP" x="16.3195" y="14.6685" smashed="yes" rot="R180">
 <attribute name="NAME" x="14.986" y="15.6845" size="0.8128" layer="25"/>
 <attribute name="VALUE" x="17.3355" y="16.0655" size="0.4064" layer="27" rot="R180"/>
 </element>
-<element name="R18" library="SparkFun-Resistors" package="0805" value="" x="38.4175" y="14.6685" smashed="yes" rot="R180">
+<element name="R18" library="SparkFun-Resistors" package="0805" value="DNP" x="38.4175" y="14.6685" smashed="yes" rot="R180">
 <attribute name="NAME" x="37.0205" y="15.6845" size="0.8128" layer="25"/>
 <attribute name="VALUE" x="39.4335" y="16.0655" size="0.4064" layer="27" rot="R180"/>
